File: ColorToSound.sch (KiCad schematic (older format))
At the start: 14 parts

Commit message: * 基本回路図の作成
Parts:
- added C?: 470u, symbol CP
- added Q?: Q_NMOS_GDS, symbol Q_NMOS_GDS
- added R? (x2): 1k, symbol R
- added R? (x8): R, symbol R
- added R?: 150, symbol R
- C? (x2): value C -> 0.1u
Connections:
- net +5V: now also C?.1, C?.1, IC?.1 (VDD), IC?.20 (VDD), R?.1, R?.1, R?.1
- net GND: now also C?.2, C?.2, IC?.19 (VSS_1), IC?.2 ((GND)(1)), IC?.3 ((GND)(2)), IC?.4 ((GND)(3)), IC?.5 (GND), IC?.7 ((GND)(4)), IC?.8 ((GND)(5)), IC?.8 (VSS), IC?.9 ((GND)(6)), LS?.2, Q?.3 (S), Q?.3 (S), Q?.3 (S), Q?.3 (S), R?.2, R?.2, R?.2, R?.2
- net at IC?.12 (RC1): now also R?.2
- net at IC?.13 (RC2): now also R?.2
- net at IC?.14 (RC3): now also IC?.6 (SCL), R?.2
- net at IC?.15 (RC4): now also IC?.10 (SDA), R?.2
- net at IC?.21 (RB0): now also R?.2
- net at IC?.26 (RB5): now also R?.2
- net at LS?.1: now also C?.2
- net at Q?.1 (G): now also R?.1, R?.1 (x3)
- new net: Q?.1 (G), R?.1, R?.1
- new net: C?.1, Q?.2 (D), R?.2
Other:
- moved on the sheet: C?, D?, IC?, LS?, Q?, R?
